File: scale.kicad_pcb (KiCad board)
At the start: 2 copper layers, 177.4 x 164.4 mm, 48 parts, among them J1 DMS, J2 SWD, J5 Display, P1 TC, Q1 s8550, Q2 AO3400, SW2 TARA, U1 HX711, U2 USBLC6-4, U3 AMS1117-3.3, U4 STM32F072CBTx, U5 QMA7981

Commit message: push
Parts:
- C1, C10, C11, C12, C13, C14, C15, C16, C17, C18, C19, C2, C3, C4, C5, C6, C7, C8, C9, D3, J1, Q1, Q2, R1, R10, R13, R14, R15, R16, R17, R2, R3, R4, R5, R6, R7, R8, R9, SW2, U1, U2, U3, U4, U5, USB1: moved to B.Cu
- J2, P1: moved to F.Cu
- moved R8 193.1 mm to (217.1, 114.2)
- moved C10 192.1 mm to (211.2, 146.6), turned to 0 degrees
- moved C19 192.1 mm to (211.2, 150.6), turned to 0 degrees
- moved R10 192.1 mm to (211.2, 145.3), turned to 0 degrees
- moved C15 191.3 mm to (210.7, 148.6)
- moved Q2 191.3 mm to (210.7, 142.8)
- moved C7 189.0 mm to (213.8, 117.0), turned to 90 degrees
- moved U2 189.0 mm to (216.3, 117.0), turned to 270 degrees
- moved USB1 189.0 mm to (220.6, 117.0), turned to 270 degrees
- moved R9 185.0 mm to (217.1, 119.7)
- moved C13 184.7 mm to (206.7, 141.7), turned to 0 degrees
- moved C9 184.1 mm to (203.7, 125.2), turned to 270 degrees
- moved C8 184.1 mm to (204.9, 125.2), turned to 270 degrees
- moved C12 183.9 mm to (203.7, 128.7), turned to 270 degrees
- moved C11 183.9 mm to (204.9, 128.7), turned to 270 degrees
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Routing:
- net HX_RATE: track 36.2 -> 12.1 mm
- net +3V3: track 101.6 -> 77.6 mm, vias 18 -> 7
- net HX_CLK: track 31.6 -> 11.3 mm
- net HX_MISO: track 33.8 -> 13.9 mm
- net D-: track 36.7 -> 20.2 mm, vias 3 -> 2
- net D+: track 37.1 -> 21.1 mm, vias 2 -> 1
- net SWDIO: track 14.0 -> 0.00 mm, vias 1 -> 0
- net LED_STATUS: track 23.1 -> 13.2 mm, vias 1 -> 0
- net Net-(R10-Pad1): track 16.7 -> 9.07 mm, vias 4 -> 3
- net VBUS: track 18.4 -> 12.8 mm
- net SWCLK: track 7.67 -> 2.77 mm
- net GND: vias 56 -> 31
Other:
- board size 177.4 x 164.4 mm -> 128 x 78.7 mm

Commit message: push
Parts:
- added J6: TOUCH, otter:Touchpad_1305_0925, F.Cu at (263.2, 118.8)
- moved J2 207.6 mm to (203.0, 105.0), turned to 270 degrees
- moved P1 197.0 mm to (189.6, 105.0)
- moved Q2 29.2 mm to (207.6, 113.8)
- moved C18 18.9 mm to (212.8, 144.0)
- moved C19 17.5 mm to (211.4, 133.1), turned to 45 degrees
- moved U5 17.5 mm to (211.8, 146.0), turned to 270 degrees
- moved C17 17.2 mm to (210.8, 148.0), turned to 0 degrees
- moved C15 16.6 mm to (209.6, 132.0), turned to 315 degrees
- moved C10 16.5 mm to (208.6, 130.2), turned to 45 degrees
- moved R10 16.3 mm to (207.7, 129.4), turned to 45 degrees
- moved R14 14.6 mm to (208.2, 143.5), turned to 225 degrees
- moved R15 14.2 mm to (209.5, 144.0), turned to 45 degrees
- moved C13 12.6 mm to (201.9, 130.0), turned to 45 degrees
- moved C14 12.5 mm to (206.5, 142.2), turned to 225 degrees
- moved U4 11.7 mm to (204.3, 135.9), turned to 225 degrees
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Connections:
- U2 pad 3: D+ -> D-
- U2 pad 4: Net-(U2-Pad4) -> D+
- U2 pad 6: D- -> Net-(U2-Pad6)
Routing:
- net D-: track 20.2 -> 73.0 mm
- net D+: track 21.1 -> 71.4 mm, vias 1 -> 0
- net SWDIO: track 0.00 -> 43.7 mm, vias 0 -> 2
- net SWCLK: track 2.77 -> 44.2 mm, vias 0 -> 1
- net IPS_PWM: track 3.81 -> 30.2 mm
- net HX_RATE: track 12.1 -> 33.2 mm, vias 0 -> 2
- net HX_CLK: track 11.3 -> 27.5 mm, vias 0 -> 2
- net HX_MISO: track 13.9 -> 30.0 mm
- net LED_STATUS: track 13.2 -> 0.00 mm
- net VBUS: track 12.8 -> 21.7 mm
- net IPS_CS: track 15.3 -> 20.4 mm, vias 1 -> 0
- net IPS_RESET: track 14.7 -> 19.3 mm, vias 1 -> 0
- net IPS_DC: track 14.0 -> 18.2 mm, vias 1 -> 0
- net IPS_SDA: track 18.8 -> 15.9 mm, vias 2 -> 0
- net ACC_SCL: track 11.5 -> 8.59 mm, vias 0 -> 2
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Other:
- outline, holes or cut-outs redrawn
- board text removed: "Schraubloch hier"

Commit message: push
Parts:
- added G***: LOGO, otter:ketaott_2120, F.Cu at (199.5, 137.5)
- moved SW2 255.0 mm to (292.3, 132.2)
- moved D3 238.7 mm to (296.4, 140.3)
- moved R13 238.7 mm to (293.4, 140.3)
- moved J6 30.8 mm to (294.0, 120.0)
- moved R16 19.4 mm to (207.2, 119.7), turned to 0 degrees
- moved R17 18.1 mm to (207.2, 120.9), turned to 180 degrees
Routing:
- net +3V3: track 74.8 -> 166.5 mm, vias 3 -> 6
- net VBUS: track 21.7 -> 25.7 mm
- net IPS_SCL: track 17.0 -> 20.8 mm
- net IPS_SDA: track 15.9 -> 19.6 mm
- net TSC_01: track 6.01 -> 3.29 mm
- net GND: track 23.2 -> 21.7 mm, vias 13 -> 83
- added copper zone on B.Cu, net GND
- added copper zone on F.Cu, net GND
- removed copper zone on F.Cu, net +3V3

Commit message: push
Parts:
- removed G***: LOGO, otter:ketaott_2120
- removed J2: SWD, Connector_PinHeader_2.54mm:PinHeader_1x04_P2.54mm_Vertical
- removed J6: TOUCH, otter:Touchpad_1305_0925
- added C20: 10u, otter:C_0603, B.Cu at (212.0, 109.0)
- added C21: 10u, otter:C_0603, B.Cu at (203.2, 108.4)
- added D1: CHARGING, LED_SMD:LED_0603_1608Metric, B.Cu at (222.0, 103.8)
- added J3: Batt, Connector_JST:JST_GH_SM02B-GHS-TB_1x02-1MP_P1.25mm_Horizontal, B.Cu at (199.6, 107.5)
- added JP1: BATT, otter:J_0603_90, B.Cu at (218.8, 122.2)
- added R11: 5k1, otter:R_0603, B.Cu at (219.0, 103.8)
- added R12: 5k1, otter:R_0603, B.Cu at (212.0, 106.6)
- added R18: 5k1, otter:R_0603, B.Cu at (208.0, 104.4)
- added R19: 5k1, otter:R_0603, B.Cu at (210.4, 104.4)
- added U6: TP4056, Package_SO:SOP-8_3.9x4.9mm_P1.27mm, B.Cu at (207.5, 107.8)
- SW2: footprint Button_Switch_SMD:SW_SPST_EVQP7C -> otter:K2-1102DP-C4SW-04; moved to F.Cu
- moved D3 81.6 mm to (214.7, 139.8)
- moved R13 81.6 mm to (211.8, 139.8)
- moved SW2 75.4 mm to (220.8, 108.4)
- moved P1 1.00 mm to (189.6, 106.0)
Connections:
- C8 pad 1: VBUS -> Net-(C8-Pad1)
- C9 pad 1: VBUS -> Net-(C8-Pad1)
- U3 pad 3: VBUS -> Net-(C8-Pad1)
Routing:
- net Net-(R10-Pad1): track 7.18 -> 59.9 mm, vias 2 -> 3
- net VBat: track 0.00 -> 40.0 mm, vias 0 -> 4
- net Net-(D1-Pad1): track 0.00 -> 24.3 mm
- net VBUS: track 25.7 -> 48.6 mm
- net +3V3: track 166.5 -> 182.7 mm, vias 6 -> 7
- net GND: track 21.7 -> 34.9 mm, vias 83 -> 86
- net SWCLK: track 44.2 -> 32.6 mm
- net SWDIO: track 43.7 -> 35.6 mm, vias 2 -> 1
- net Net-(C8-Pad1): track 0.00 -> 6.02 mm
- net LED_STATUS: track 0.00 -> 4.26 mm
- net Net-(R18-Pad2): track 0.00 -> 2.54 mm
- net Net-(R12-Pad1): track 0.00 -> 2.40 mm
- net Net-(D1-Pad2): track 0.00 -> 1.46 mm
Other:
- board text removed: "3.3V DIO GND CLK"
