File: scale.kicad_pcb (KiCad board)
At the start: 2 copper layers, 128 x 78.7 mm, 57 parts, among them J1 DMS, J3 Batt, J5 Display, P1 TC, Q1 s8550, Q2 AO3400, SW2 TARA, U1 HX711, U2 USBLC6-4, U3 AMS1117-3.3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

Commit message: pushed latest files
Routing:
- net TSC_02: track 0.00 -> 25.1 mm, vias 0 -> 3
- net TSC_01: track 3.29 -> 16.3 mm, vias 0 -> 1
- net GND: vias 86 -> 85
- added copper zone on F.Cu, net TSC_01
- added copper zone on F.Cu, net TSC_02
Changed lines of the file:
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@@
     (thickness 1.6)
     (drawings 197)
-    (tracks 560)
+    (tracks 573)
     (zones 0)
     (modules 57)
@@
   )
   (setup
-    (last_trace_width 0.2)
+    (last_trace_width 0.25)
     (user_trace_width 0.127)
     (user_trace_width 0.2)
@@
   (segment (start 214.8 126.700001) (end 214.8 126.100001) (width 0.5) (layer B.Cu) (net 6))
   (via (at 213.6 145) (size 0.6) (drill 0.4) (layers F.Cu B.Cu) (net 6))
-  (via (at 213.2 145.6) (size 0.6) (drill 0.4) (layers F.Cu B.Cu) (net 6))
   (via (at 215 144.4) (size 0.6) (drill 0.4) (layers F.Cu B.Cu) (net 6))
   (via (at 215 142.4) (size 0.6) (drill 0.4) (layers F.Cu B.Cu) (net 6))
@@
   (segment (start 220.525 114.575) (end 220.55 114.55) (width 0.5) (layer B.Cu) (net 8))
   (segment (start 219.125 114.575) (end 220.525 114.575) (width 0.5) (layer B.Cu) (net 8))
-  (segment (start 217.45 124.599998) (end 217.9 125.05) (width 0.5) (layer B.Cu) (net 69))
-  (segment (start 214.800001 124.6) (end 217.45 124.599998) (width 0.5) (layer B.Cu) (net 69))
   (segment (start 222.1 118.825) (end 221.575 119.35) (width 0.3) (layer B.Cu) (net 8))
   (segment (start 221.575 119.35) (end 220.55 119.35) (width 0.3) (layer B.Cu) (net 8))
@@
   (segment (start 205.47 105.845) (end 204.875 105.845) (width 0.5) (layer B.Cu) (net 8))
   (segment (start 209.28 109.655) (end 205.47 105.845) (width 0.5) (layer B.Cu) (net 8))
-  (segment (start 218.249999 125.050001) (end 217.9 125.050001) (width 0.5) (layer B.Cu) (net 69))
   (segment (start 208.101219 130.843146) (end 208.030509 130.772435) (width 0.2) (layer B.Cu) (net 9))
   (segment (start 208.10122 132.469491) (end 208.101219 130.843146) (width 0.2) (layer B.Cu) (net 9))
@@
   (segment (start 220.55 116.2) (end 219.192831 116.2) (width 0.2) (layer B.Cu) (net 29))
   (via (at 219.042841 116.05001) (size 0.6) (drill 0.4) (layers F.Cu B.Cu) (net 29))
-  (segment (start 221.475 116.7) (end 220.55 116.7) (width 0.2) (layer B.Cu) (net 30))
-  (segment (start 221.575001 116.800001) (end 221.475 116.7) (width 0.2) (layer B.Cu) (net 30))
-  (segment (start 221.575001 117.599999) (end 221.575001 116.800001) (width 0.2) (layer B.Cu) (net 30))
-  (segment (start 221.475 117.7) (end 221.575001 117.599999) (width 0.2) (layer B.Cu) (net 30))
-  (segment (start 220.55 117.7) (end 221.475 117.7) (width 0.2) (layer B.Cu) (net 30))
   (segment (start 217.25 116) (end 217.25 115.85) (width 0.2) (layer B.Cu) (net 29))
   (via (at 219.02531 117.27531) (size 0.6) (drill 0.4) (layers F.Cu B.Cu) (net 29))
@@
   (segment (start 218.25 116.75) (end 217.25 116.75) (width 0.2) (layer B.Cu) (net 29))
   (segment (start 218.94999 116.05001) (end 218.25 116.75) (width 0.2) (layer B.Cu) (net 29))
+  (segment (start 221.475 116.7) (end 220.55 116.7) (width 0.2) (layer B.Cu) (net 30))
+  (segment (start 221.575001 116.800001) (end 221.475 116.7) (width 0.2) (layer B.Cu) (net 30))
+  (segment (start 221.575001 117.599999) (end 221.575001 116.800001) (width 0.2) (layer B.Cu) (net 30))
+  (segment (start 221.475 117.7) (end 221.575001 117.599999) (width 0.2) (layer B.Cu) (net 30))
+  (segment (start 220.55 117.7) (end 221.475 117.7) (width 0.2) (layer B.Cu) (net 30))
   (segment (start 220.55 116.7) (end 218.855313 116.7) (width 0.2) (layer B.Cu) (net 30))
   (segment (start 217.25 118.05) (end 217.25 117.32) (width 0.2) (layer B.Cu) (net 30))
@@
   (segment (start 209.16188 133.530152) (end 210.788224 133.530152) (width 0.2) (layer B.Cu) (net 64))
   (segment (start 208.498967 134.193064) (end 209.16188 133.530152) (width 0.2) (layer B.Cu) (net 64))
+  (segment (start 210.6 136.294097) (end 210.6 137.4) (width 0.127) (layer B.Cu) (net 66))
+  (via (at 208.8 139.2) (size 0.6) (drill 0.4) (layers F.Cu B.Cu) (net 66))
+  (segment (start 210.6 137.4) (end 208.8 139.2) (width 0.127) (layer B.Cu) (net 66))
+  (via (at 204.8 143) (size 0.6) (drill 0.4) (layers F.Cu B.Cu) (net 66))
+  (segment (start 208.8 139.2) (end 205 143) (width 0.127) (layer F.Cu) (net 66))
+  (segment (start 205 143) (end 204.8 143) (width 0.127) (layer F.Cu) (net 66))
+  (via (at 195.8 153.2) (size 0.6) (drill 0.4) (layers F.Cu B.Cu) (net 66))
+  (segment (start 204.8 143) (end 195.8 152) (width 0.127) (layer B.Cu) (net 66))
+  (segment (start 195.8 152) (end 195.8 153.2) (width 0.127) (layer B.Cu) (net 66))
+  (segment (start 209.206074 134.900171) (end 210.6 136.294097) (width 0.127) (layer B.Cu) (net 66))
   (segment (start 209.463814 133.935324) (end 210.168092 133.935324) (width 0.127) (layer B.Cu) (net 67))
   (segment (start 208.852521 134.546618) (end 209.463814 133.935324) (width 0.127) (layer B.Cu) (net 67))
   (segment (start 210.168092 133.935324) (end 210.858936 134.626167) (width 0.127) (layer B.Cu) (net 67))
   (segment (start 210.858936 134.626167) (end 211.601398 134.626167) (width 0.127) (layer B.Cu) (net 67))
+  (segment (start 211.601398 134.626167) (end 213.826167 134.626167) (width 0.127) (layer B.Cu) (net 67))
+  (segment (start 213.826167 134.626167) (end 218.8 139.6) (width 0.127) (layer B.Cu) (net 67))
+  (via (at 218.8 143.4) (size 0.6) (drill 0.4) (layers F.Cu B.Cu) (net 67))
+  (segment (start 218.8 139.6) (end 218.8 143.4) (width 0.127) (layer B.Cu) (net 67))
+  (segment (start 217.45 124.599998) (end 217.9 125.05) (width 0.5) (layer B.Cu) (net 69))
+  (segment (start 214.800001 124.6) (end 217.45 124.599998) (width 0.5) (layer B.Cu) (net 69))
+  (segment (start 218.249999 125.050001) (end 217.9 125.050001) (width 0.5) (layer B.Cu) (net 69))
   (segment (start 218.7125 124.237501) (end 217.9 125.050001) (width 0.5) (layer B.Cu) (net 69))
   (segment (start 218.7125 123) (end 218.7125 124.237501) (width 0.5) (layer B.Cu) (net 69))
@@
       )
     )
+  )
+  (zone (net 66) (net_name TSC_02) (layer F.Cu) (hatch edge 0.508)
+    (connect_pads (clearance 0.1))
+    (min_thickness 0.254)
+    (fill yes (arc_segments 32) (thermal_gap 0.508) (thermal_bridge_width 0.508) (smoothing fillet) (radius 0.2))
+    (polygon
+      (pts
+        (xy 204.6 157.6) (xy 204.6 167.6) (xy 196 172.6) (xy 187.2 167.6) (xy 187.2 157.6)
+        (xy 195.8 152.6)
+      )
+    )
+  )
+  (zone (net 67) (net_name TSC_01) (layer F.Cu) (hatch edge 0.508)
+    (priority 1)
+    (connect_pads (clearance 0.1))
+    (min_thickness 0.254)
+    (fill yes (arc_segments 32) (thermal_gap 0.508) (thermal_bridge_width 0.508) (smoothing fillet) (radius 0.2))
+    (polygon
+      (pts
+        (xy 224.4 146) (xy 224.4 152.8) (xy 218.8 156.2) (xy 213 152.8) (xy 213 146)
+        (xy 218.8 142.6)
+      )
+    )

Commit message: initial commit
Parts:
- removed D3: STATUS, LED_SMD:LED_0603_1608Metric
- removed R16, R17: 5k1, otter:R_0603
- added C22: DNP, otter:C_0603, B.Cu at (183.2, 149.2)
- added C23: DNP, otter:C_0603, B.Cu at (184.4, 149.2)
- added D2: CHARGING, otter:BL-HUB34E-AV-TRB, B.Cu at (222.3, 103.8)
- added JP2: B, otter:J_0603_90, B.Cu at (187.0, 132.2)
- added JP3: B, otter:J_0603_90, B.Cu at (184.2, 132.2)
- C18: value 10u -> 100n
- C2: value 1u -> 10u
- D1: value CHARGING -> STATUS; footprint LED_SMD:LED_0603_1608Metric -> otter:BL-HUB34E-AV-TRB
- R3: value 0 -> 100
- R4: value 0 -> 0.5; footprint otter:R_0603 -> otter:R_0805
- U5: value QMA7981 -> BMA280
- moved R4 44.1 mm to (213.9, 111.4), turned to 135 degrees
- moved R3 39.8 mm to (209.9, 114.8), turned to 90 degrees
- moved D1 38.5 mm to (223.9, 142.3)
- moved C17 5.85 mm to (209.9, 142.2), turned to 135 degrees
- moved U5 2.52 mm to (212.3, 143.6), turned to 0 degrees
- moved C2 1.82 mm to (179.9, 133.8)
- moved C18 1.57 mm to (214.2, 143.6), turned to 270 degrees
- moved R13 0.94 mm to (210.9, 139.3)
- moved C1 0.86 mm to (179.9, 132.7)
- moved R15 0.63 mm to (208.9, 143.8)
- moved R14 0.50 mm to (207.9, 143.1)
Connections:
- net LED_ERR renamed Net-(U4-Pad18)
- C20 pad 1: VBUS -> Net-(C20-Pad1)
- D1 pad 1: Net-(D1-Pad1) -> GND
- J5 pad 12: +3V3 -> Net-(J5-Pad12)
- R11 pad 1: VBUS -> Net-(C20-Pad1)
- R11 pad 2: Net-(D1-Pad2) -> Net-(D2-Pad2)
- R13 pad 2: Net-(D3-Pad2) -> Net-(D1-Pad2)
- R18 pad 1: VBUS -> Net-(C20-Pad1)
- R3 pad 1: Net-(R3-Pad1) -> +3V3
- R3 pad 2: GND -> Net-(J5-Pad12)
- R4 pad 1: Net-(R4-Pad1) -> VBUS
- R4 pad 2: GND -> Net-(C20-Pad1)
- U1 pad 10: Net-(R3-Pad1) -> Net-(JP2-Pad2)
- U1 pad 14: GND -> HX_XO
- U1 pad 9: Net-(R4-Pad1) -> Net-(JP3-Pad2)
- U4 pad 14: HX_RATE -> Net-(U4-Pad14)
- U4 pad 15: HX_CLK -> Net-(U4-Pad15)
- U4 pad 16: HX_MISO -> Net-(U4-Pad16)
- U4 pad 17: HX_MISO -> LED_STATUS
- U4 pad 19: LED_STATUS -> INT2
- U4 pad 20: Net-(U4-Pad20) -> INT1
- U4 pad 25: Net-(U4-Pad25) -> HX_RATE
- U4 pad 26: Net-(U4-Pad26) -> HX_CLK
- U4 pad 27: Net-(U4-Pad27) -> HX_MISO
- U4 pad 28: Net-(U4-Pad28) -> HX_MISO
- U4 pad 29: Net-(U4-Pad29) -> HX_XO
- U4 pad 38: IPS_PWM -> IPS_RESET
- U4 pad 39: IPS_CS -> IPS_SCL
- U4 pad 40: IPS_RESET -> Net-(U4-Pad40)
- U4 pad 41: IPS_DC -> IPS_SDA
- U4 pad 42: IPS_SCL -> IPS_DC
- U4 pad 43: IPS_SDA -> IPS_CS
- U4 pad 45: Net-(U4-Pad45) -> IPS_PWM
- U5 pad 10: +3V3 -> Net-(U5-Pad10)
- U5 pad 11: Net-(U5-Pad11) -> +3V3
- U5 pad 4: GND -> Net-(U5-Pad4)
- U5 pad 5: Net-(U5-Pad5) -> INT1
- U5 pad 6: Net-(U5-Pad6) -> INT2
- U6 pad 4: VBUS -> Net-(C20-Pad1)
- U6 pad 7: Net-(D1-Pad1) -> Net-(D2-Pad1)
- U6 pad 8: VBUS -> Net-(C20-Pad1)
Routing:
- net Net-(D2-Pad1): track 0.00 -> 26.5 mm
- net VBUS: track 48.6 -> 24.2 mm
- net Net-(D1-Pad1): track 24.3 -> 0.00 mm
- net HX_XO: track 0.00 -> 23.7 mm, vias 0 -> 2
- net Net-(C20-Pad1): track 0.00 -> 22.8 mm
- net +3V3: track 182.7 -> 164.3 mm, vias 7 -> 9
- net Net-(JP3-Pad2): track 0.00 -> 16.7 mm
- net Net-(JP2-Pad2): track 0.00 -> 11.8 mm
- net Net-(D1-Pad2): track 1.46 -> 12.4 mm, vias 0 -> 2
- net INT2: track 0.00 -> 7.43 mm
- net Net-(J5-Pad12): track 0.00 -> 7.29 mm
- net HX_CLK: track 27.5 -> 20.4 mm
- net INT1: track 0.00 -> 7.13 mm
- net HX_MISO: track 30.0 -> 22.9 mm
- net HX_RATE: track 33.2 -> 26.7 mm, vias 2 -> 0
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Other:
- board text added: "C"
