File: scale.sch (KiCad schematic (older format))
At the start: 51 parts, among them J1 DMS, J2 SWD, J3 DMS, J4 DMS, J5 Display, J6 TOUCH, P1 TC, Q1 s8550, Q2 AO3400, SW2 TARA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

Commit message: push
Parts:
- removed J3, J4: DMS, MountingHole:MountingHole_3.2mm_M3_Pad, symbol Connector:Screw_Terminal_01x01
Changed lines of the file:
@@
 	4350 1650 4350 1600
-$Comp
-L Connector:Screw_Terminal_01x01 J3
-U 1 1 5E732E49
-P 7650 4000
-F 0 "J3" H 7730 4042 50  0000 L CNN
-F 1 "DMS" H 7730 3951 50  0000 L CNN
-F 2 "MountingHole:MountingHole_3.2mm_M3_Pad" H 7650 4000 50  0001 C CNN
-F 3 "~" H 7650 4000 50  0001 C CNN
-	1    7650 4000
-	1    0    0    -1
-$EndComp
-$Comp
-L Connector:Screw_Terminal_01x01 J4
-U 1 1 5E7349A0
-P 7650 4200
-F 0 "J4" H 7730 4242 50  0000 L CNN
-F 1 "DMS" H 7730 4151 50  0000 L CNN
-F 2 "MountingHole:MountingHole_3.2mm_M3_Pad" H 7650 4200 50  0001 C CNN
-F 3 "~" H 7650 4200 50  0001 C CNN
-	1    7650 4200
-	1    0    0    -1
-$EndComp
-$Comp
-L power:GND #PWR0141
-U 1 1 5E7380DC
-P 7450 4000
-F 0 "#PWR0141" H 7450 3750 50  0001 C CNN
-F 1 "GND" V 7455 3872 50  0000 R CNN
-F 2 "" H 7450 4000 50  0001 C CNN
-F 3 "" H 7450 4000 50  0001 C CNN
-	1    7450 4000
-	0    1    1    0
-$EndComp
-$Comp
-L power:GND #PWR0142
-U 1 1 5E738A77
-P 7450 4200
-F 0 "#PWR0142" H 7450 3950 50  0001 C CNN
-F 1 "GND" V 7455 4072 50  0000 R CNN
-F 2 "" H 7450 4200 50  0001 C CNN
-F 3 "" H 7450 4200 50  0001 C CNN
-	1    7450 4200
-	0    1    1    0
-$EndComp
 $Comp
 L Connector_Generic:Conn_01x13 J5

Commit message: push
Connections:
- net D+: now also U2.4 (IO3); no longer U2.3 (IO2)
- net D-: now also U2.3 (IO2); no longer U2.6 (IO4)
Changed lines of the file:
@@
 	1    0    0    -1
 $EndComp
+Text GLabel 1950 4150 2    50   Input ~ 0
+D+
 Text GLabel 1350 4050 0    50   Input ~ 0
-D+
-Text GLabel 1950 4050 2    50   Input ~ 0
 D-
 $Comp

Commit message: push
Parts:
- added J?: Conn_01x02_Male, symbol Connector:Conn_01x02_Male
- added JP?: BATT, symbol Jumper:Jumper_3_Bridged12
- added R?: 5k1, otter:R_0603, symbol Device:R_Small
- added U?: TP4056, symbol otter:TP4056
Connections:
- net GND: now also R?.2, U?.3 (GND)
- net VBUS: now also JP?.1 (A), U?.4 (VCC), U?.8 (CE); no longer C8.1, C9.1, U3.3 (VI)
- new net: R?.1, U?.2 (PROG)
- new net: C8.1, C9.1, JP?.2 (C), U3.3 (VI)
- new net VBat: JP?.3 (B)
- no-connect marks 7 -> 9
Other:
- note added: "TODO:\nBatt\nLED\nButton"
Changed lines of the file:
@@
 L power:VBUS #PWR0138
 U 1 1 5E6D26A8
-P 3450 1250
-F 0 "#PWR0138" H 3450 1100 50  0001 C CNN
-F 1 "VBUS" V 3465 1378 50  0000 L CNN
-F 2 "" H 3450 1250 50  0001 C CNN
-F 3 "" H 3450 1250 50  0001 C CNN
-	1    3450 1250
-	0    -1   -1   0
+P 3300 1500
+F 0 "#PWR0138" H 3300 1350 50  0001 C CNN
+F 1 "VBUS" V 3315 1628 50  0000 L CNN
+F 2 "" H 3300 1500 50  0001 C CNN
+F 3 "" H 3300 1500 50  0001 C CNN
+	1    3300 1500
+	-1   0    0    1
 $EndComp
 $Comp
@@
 Wire Wire Line
 	6700 1950 6700 2150
+$Comp
+L otter:TP4056 U?
+U 1 1 5E69DFD2
+P 10200 4100
+F 0 "U?" H 10200 4515 50  0000 C CNN
+F 1 "TP4056" H 10200 4424 50  0000 C CNN
+F 2 "" H 10200 4100 50  0001 C CNN
+F 3 "" H 10200 4100 50  0001 C CNN
+	1    10200 4100
+	1    0    0    -1
+$EndComp
+$Comp
+L Jumper:Jumper_3_Bridged12 JP?
+U 1 1 5E6B4A0A
+P 3300 1250
+F 0 "JP?" V 3346 1317 50  0000 L CNN
+F 1 "BATT" V 3255 1317 50  0000 L CNN
+F 2 "" H 3300 1250 50  0001 C CNN
+F 3 "~" H 3300 1250 50  0001 C CNN
+	1    3300 1250
+	0    -1   -1   0
+$EndComp
+$Comp
+L power:VBUS #PWR?
+U 1 1 5E6BE96C
+P 9600 3950
+F 0 "#PWR?" H 9600 3800 50  0001 C CNN
+F 1 "VBUS" V 9615 4078 50  0000 L CNN
+F 2 "" H 9600 3950 50  0001 C CNN
+F 3 "" H 9600 3950 50  0001 C CNN
+	1    9600 3950
+	0    -1   -1   0
+$EndComp
+Text GLabel 3300 1000 1    50   Input ~ 0
+VBat
+Text Notes 7850 -650 0    50   ~ 0
+TODO:\nBatt\nLED\nButton
+Wire Wire Line
+	9800 4050 9700 4050
+Wire Wire Line
+	9700 4050 9700 3950
+Wire Wire Line
+	9700 3950 9600 3950
+Wire Wire Line
+	9700 3950 9800 3950
+Connection ~ 9700 3950
+$Comp
+L Device:R_Small R?
+U 1 1 5E6F63E6
+P 10900 4350
+F 0 "R?" V 11004 4350 50  0000 C CNN
+F 1 "5k1" V 10900 4350 50  0000 C CNN
+F 2 "otter:R_0603" H 10900 4350 50  0001 C CNN
+F 3 "~" H 10900 4350 50  0001 C CNN
+	1    10900 4350
+	1    0    0    -1
+$EndComp
+$Comp
+L power:GND #PWR?
+U 1 1 5E6F63EC
+P 10900 4450
+F 0 "#PWR?" H 10900 4200 50  0001 C CNN
+F 1 "GND" H 10905 4277 50  0000 C CNN
+F 2 "" H 10900 4450 50  0001 C CNN
+F 3 "" H 10900 4450 50  0001 C CNN
+	1    10900 4450
+	1    0    0    -1
+$EndComp
+Wire Wire Line
+	10600 4150 10900 4150
+Wire Wire Line
+	10900 4150 10900 4250
+$Comp
+L power:GND #PWR?
+U 1 1 5E6FEDCB
+P 10700 4450
+F 0 "#PWR?" H 10700 4200 50  0001 C CNN
+F 1 "GND" H 10705 4277 50  0000 C CNN
+F 2 "" H 10700 4450 50  0001 C CNN
+F 3 "" H 10700 4450 50  0001 C CNN
+	1    10700 4450
+	1    0    0    -1
+$EndComp
+Wire Wire Line
+	10700 4450 10700 4250
+Wire Wire Line
+	10700 4250 10600 4250
+NoConn ~ 9800 4150
+NoConn ~ 9800 4250
+$Comp
+L Connector:Conn_01x02_Male J?
+U 1 1 5E70FE29
+P 11350 4050
+F 0 "J?" H 11322 3932 50  0000 R CNN
+F 1 "Conn_01x02_Male" H 11322 4023 50  0000 R CNN
+F 2 "" H 11350 4050 50  0001 C CNN
+F 3 "~" H 11350 4050 50  0001 C CNN
+	1    11350 4050
+	-1   0    0    1
+$EndComp
 $EndSCHEMATC

Commit message: push
Parts:
- removed J2: SWD, Connector_PinHeader_2.54mm:PinHeader_1x04_P2.54mm_Vertical, symbol Connector:Conn_01x04_Female
- added C20, C21: 10u, otter:C_0603, symbol Device:C_Small
- added D1: CHARGING, LED_SMD:LED_0603_1608Metric, symbol Device:LED
- added R11, R18, R19: 5k1, otter:R_0603, symbol Device:R_Small
- J3: renamed from J?; value Conn_01x02_Male -> Batt; footprint (none) -> Connector_JST:JST_GH_SM02B-GHS-TB_1x02-1MP_P1.25mm_Horizontal; symbol Connector:Conn_01x02_Male -> Connector_Generic_MountingPin:Conn_01x02_MountingPin
- JP1: renamed from JP?; footprint (none) -> otter:J_0603_90
- SW2: footprint Button_Switch_SMD:SW_SPST_EVQP7C -> otter:K2-1102DP-C4SW-04
- U6: renamed from U?; footprint (none) -> Package_SO:SOP-8_3.9x4.9mm_P1.27mm
- gave numbers to parts that had none: 1
Connections:
- net GND: now also J3.2 (Pin_2), J3.MP (MountPin), C20.2, C21.2, R19.2
- net VBUS: now also C20.1, R11.1, R18.1
- net VBat: now also J3.1 (Pin_1), U6.5 (BAT), C21.1
- net at U6.1 (TEMP): now also R18.2, R19.1
- net at U6.7 (\CHRG): now also D1.1 (K)
- new net: D1.2 (A), R11.2
- no-connect marks 9 -> 8
Other:
- note added: "TODO:\nLED"
- note removed: "TODO:\nBatt\nLED\nButton"
- moved on the sheet: D3, R12, R13, R14, R15, R16, R17, U6

Commit message: initial commit
Parts:
- removed D1: CHARGING, LED_SMD:LED_0603_1608Metric, symbol Device:LED
- removed D3: STATUS, LED_SMD:LED_0603_1608Metric, symbol Device:LED
- removed J6: TOUCH, otter:Touchpad_1305_0925, symbol Connector:Screw_Terminal_01x01
- removed R16, R17: 5k1, otter:R_0603, symbol Device:R_Small
- removed U5: QMA7981, Package_LGA:LGA-12_2x2mm_P0.5mm, symbol otter:QMA7981
- added C22, C23: DNP, otter:C_0603, symbol Device:C_Small
- added D1: STATUS, otter:BL-HUB34E-AV-TRB, symbol Device:LED_PAD
- added D2: CHARGING, otter:BL-HUB34E-AV-TRB, symbol Device:LED_PAD
- added JP2, JP3: B, otter:J_0603_90, symbol Jumper:Jumper_3_Bridged12
- added U5: BMA280, Package_LGA:LGA-12_2x2mm_P0.5mm, symbol otter:BMA280
- C18: value 10u -> 100n
- C2: value 1u -> 10u
- R3: value 0 -> 100
- R4: value 0 -> 0.5; footprint otter:R_0603 -> otter:R_0805
Connections:
- net +3V3: now also R3.1, C22.1, C23.1, U5.11 (PS), U5.3 (VDDIO), U5.7 (VDD); no longer J5.12 (Pin_12)
- net ACC_SCL: now also U5.12 (SCx)
- net ACC_SDA: now also U5.2 (SDx)
- net GND: now also C22.2, C23.2, D1.1 (K), JP2.1 (A), JP3.1 (A), U5.1 (SDO), U5.8 (GNDIO), U5.9 (GND); no longer R3.2, R4.2, U1.14 (XI)
- net HX_CLK: now also U4.26 (PB13); no longer U4.15 (PA5)
- net HX_MISO: now also U4.27 (PB14), U4.28 (PB15); no longer U4.16 (PA6), U4.17 (PA7)
- net HX_RATE: now also U4.25 (PB12); no longer U4.14 (PA4)
- net IPS_CS: now also U4.43 (PB7); no longer U4.39 (PB3)
- net IPS_DC: now also U4.42 (PB6); no longer U4.41 (PB5)
- net IPS_PWM: now also U4.45 (PB8); no longer U4.38 (PA15)
- net IPS_RESET: now also U4.38 (PA15); no longer U4.40 (PB4)
- net IPS_SCL: now also U4.39 (PB3); no longer U4.42 (PB6)
- net IPS_SDA: now also U4.41 (PB5); no longer U4.43 (PB7)
- net LED_STATUS: now also U4.17 (PA7); no longer U4.19 (PB1)
- net VBUS: now also R4.1; no longer C20.1, R11.1, R18.1, U6.4 (VCC), U6.8 (CE)
- net at U1.10 (INPB): now also JP2.2 (C); no longer R3.1
- net at U1.9 (INNB): now also JP3.2 (C); no longer R4.1
- net at J1.4 (Pin_4), R1.2: now also JP2.3 (B)
- net at J1.3 (Pin_3), R2.2: now also JP3.3 (B)
- net INT1: now reaches U4.20 (PB2)
- net INT1: now also U5.5 (INT1)
- net HX_XO: now reaches U4.29 (PA8)
- net HX_XO: now also U1.14 (XI)
- net at U6.7 (\CHRG): now also D2.1 (K)
- net at R11.2: now also D2.2 (A)
- net at R13.2: now also D1.2 (A)
- net LED_ERR: no longer names the net of U4.18 (PB0)
- new net: C20.1, R11.1, R18.1, R4.2, U6.4 (VCC), U6.8 (CE)
- new net: J5.12 (Pin_12), R3.2
- new net INT2: U4.19 (PB1), U5.6 (INT2)
Other:
- note added: "TODO:\n"
- note removed: "TODO:\nLED"
- moved on the sheet: C20
